File: Electronics/heating-controller.brd (EAGLE design)
At the start: 60 x 61.6 mm, 25 parts, among them IC1 AP1117 (3v3), Q1 IRLB8721PBF

Commit message: Smaller 3v3 reg used, that can also stand 20V.
Parts:
- IC1: value AP1117 (3v3) -> TS2950-3v3; device v-reg:79XXS -> v-reg:TO92
- moved IC1 3.24 mm to (7.62, 37.5)
- moved R2 1.27 mm to (16.5, 47.6)
- moved C1 0.90 mm to (6.35, 26.7)
Connections:
- net +12V: now also IC1.3, JP3.7; no longer IC1.OUT
- net GND: now also IC1.2; no longer IC1.GND
- net VCC: now also IC1.1; no longer IC1.IN, JP3.7
Routing:
- net +12V: track 83.3 -> 100.0 mm, vias 0 -> 2
- net N$3: track 77.4 -> 73.3 mm
- net GND: track 130.6 -> 134.5 mm
- net VCC: track 117.1 -> 119.9 mm
- net N$5: track 7.29 -> 6.02 mm
