File: Electronics/heating-controller.sch (EAGLE design)
At the start: 19 parts, among them IC1 AP1117T33L-U, Q1 IRLB8721PBF

Commit message: First version of PCB complete.
Parts:
- added H1, H2, H3, H4: MOUNT-PAD-ROUND2.8, holes:MOUNT-PAD-ROUND2.8
- IC1: value AP1117T33L-U -> AP1117 (3v3); device v-reg:78XXS -> v-reg:79XXS
Connections:
- removed net N$13: C4.2, JP2.1
- new net N$8: C4.1, JP2.2
- net +12V: now also IC1.OUT; no longer IC1.IN
- net N$12: now also JP2.1; no longer C4.1
- net N$14: now also C4.2; no longer JP2.2
- net VCC: now also IC1.IN; no longer IC1.OUT
Other:
- moved on the sheet: C4, IC1
Changed lines of the file:
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@@
 <part name="P+7" library="supply1" deviceset="VCC" device=""/>
 <part name="Q1" library="transistor-power" deviceset="PMOSFET_N" device="TO220BV" value="IRLB8721PBF"/>
-<part name="IC1" library="v-reg" deviceset="78XXS" device="" value="AP1117T33L-U"/>
+<part name="H1" library="holes" deviceset="MOUNT-PAD-ROUND" device="2.8"/>
+<part name="H2" library="holes" deviceset="MOUNT-PAD-ROUND" device="2.8"/>
+<part name="H3" library="holes" deviceset="MOUNT-PAD-ROUND" device="2.8"/>
+<part name="H4" library="holes" deviceset="MOUNT-PAD-ROUND" device="2.8"/>
+<part name="GND10" library="supply1" deviceset="GND" device=""/>
+<part name="IC1" library="v-reg" deviceset="79XXS" device="" value="AP1117 (3v3)"/>
 </parts>
 <sheets>
@@
 <instance part="JP1" gate="A" x="7.62" y="30.48"/>
 <instance part="GND6" gate="1" x="-10.16" y="35.56"/>
-<instance part="C4" gate="G$1" x="22.86" y="17.78" rot="R90"/>
+<instance part="C4" gate="G$1" x="43.18" y="17.78" rot="R90"/>
 <instance part="JP2" gate="G$1" x="35.56" y="20.32" rot="R90"/>
 <instance part="P+6" gate="1" x="-22.86" y="30.48"/>
@@
 <instance part="P+7" gate="VCC" x="73.66" y="40.64" rot="R270"/>
 <instance part="Q1" gate="G$1" x="99.06" y="10.16"/>
-<instance part="IC1" gate="1" x="-12.7" y="81.28"/>
+<instance part="H1" gate="G$1" x="27.94" y="99.06"/>
+<instance part="H2" gate="G$1" x="35.56" y="99.06"/>
+<instance part="H3" gate="G$1" x="27.94" y="91.44"/>
+<instance part="H4" gate="G$1" x="35.56" y="91.44"/>
+<instance part="GND10" gate="1" x="20.32" y="96.52"/>
+<instance part="IC1" gate="1" x="-12.7" y="81.28" rot="R180"/>
 </instances>
 <busses>
@@
 <wire x1="-22.86" y1="86.36" x2="-22.86" y2="81.28" width="0.1524" layer="91"/>
 <junction x="-22.86" y="81.28"/>
-<pinref part="IC1" gate="1" pin="IN"/>
+<pinref part="IC1" gate="1" pin="OUT"/>
 </segment>
 <segment>
@@
 <pinref part="Q1" gate="G$1" pin="S"/>
 </segment>
+<segment>
+<pinref part="GND10" gate="1" pin="GND"/>
+<wire x1="20.32" y1="99.06" x2="27.94" y2="99.06" width="0.1524" layer="91"/>
+<wire x1="27.94" y1="99.06" x2="27.94" y2="91.44" width="0.1524" layer="91"/>
+<wire x1="27.94" y1="91.44" x2="35.56" y2="91.44" width="0.1524" layer="91"/>
+<wire x1="35.56" y1="91.44" x2="35.56" y2="99.06" width="0.1524" layer="91"/>
+</segment>
 </net>
 <net name="N$4" class="0">
@@
 <pinref part="C5" gate="G$1" pin="2"/>
 <junction x="0" y="81.28"/>
-<pinref part="IC1" gate="1" pin="OUT"/>
+<pinref part="IC1" gate="1" pin="IN"/>
 </segment>
 <segment>
@@
 <wire x1="5.08" y1="25.4" x2="17.78" y2="25.4" width="0.1524" layer="91"/>
 <wire x1="17.78" y1="25.4" x2="17.78" y2="17.78" width="0.1524" layer="91"/>
-<pinref part="C4" gate="G$1" pin="1"/>
-<wire x1="17.78" y1="17.78" x2="20.32" y2="17.78" width="0.1524" layer="91"/>
-</segment>
-</net>
-<net name="N$13" class="0">
-<segment>
-<pinref part="C4" gate="G$1" pin="2"/>
 <pinref part="JP2" gate="G$1" pin="1"/>
-<wire x1="27.94" y1="17.78" x2="33.02" y2="17.78" width="0.1524" layer="91"/>
+<wire x1="17.78" y1="17.78" x2="33.02" y2="17.78" width="0.1524" layer="91"/>
 </segment>
 </net>
 <net name="N$14" class="0">
 <segment>
-<pinref part="JP2" gate="G$1" pin="2"/>
-<wire x1="35.56" y1="17.78" x2="66.04" y2="17.78" width="0.1524" layer="91"/>
 <pinref part="U$1" gate="G$1" pin="RST"/>
 <wire x1="66.04" y1="17.78" x2="66.04" y2="38.1" width="0.1524" layer="91"/>
+<pinref part="C4" gate="G$1" pin="2"/>
+<wire x1="48.26" y1="17.78" x2="66.04" y2="17.78" width="0.1524" layer="91"/>
 </segment>
 </net>
@@
 </segment>
 </net>
+<net name="N$8" class="0">
+<segment>
+<pinref part="C4" gate="G$1" pin="1"/>
+<pinref part="JP2" gate="G$1" pin="2"/>
+<wire x1="40.64" y1="17.78" x2="35.56" y2="17.78" width="0.1524" layer="91"/>
+</segment>
+</net>
