File: Electronics/heating-controller.sch (EAGLE design)
At the start: 25 parts, among them IC1 AP1117 (3v3), Q1 IRLB8721PBF

Commit message: Smaller 3v3 reg used, that can also stand 20V.
Parts:
- IC1: value AP1117 (3v3) -> TS2950-3v3; device v-reg:79XXS -> v-reg:LP2950ACZ-3.0
Connections:
- net +12V: now also IC1.IN, JP3.7; no longer IC1.OUT
- net VCC: now also IC1.OUT; no longer IC1.IN, JP3.7
Changed lines of the file:
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@@
 <part name="R2" library="rcl" deviceset="R-EU_" device="0207/7" value="1K"/>
 <part name="R3" library="rcl" deviceset="R-EU_" device="0207/7" value="220R"/>
-<part name="GND1" library="supply1" deviceset="GND" device=""/>
 <part name="GND2" library="supply1" deviceset="GND" device=""/>
 <part name="P+1" library="supply1" deviceset="+12V" device=""/>
@@
 <part name="H4" library="holes" deviceset="MOUNT-PAD-ROUND" device="2.8"/>
 <part name="GND10" library="supply1" deviceset="GND" device=""/>
-<part name="IC1" library="v-reg" deviceset="79XXS" device="" value="AP1117 (3v3)"/>
 <part name="B1" library="rectifier" deviceset="B-DIL" device=""/>
-<part name="P+8" library="supply1" deviceset="VCC" device=""/>
 <part name="GND11" library="supply1" deviceset="GND" device=""/>
 <part name="JP3" library="pinhead" deviceset="PINHD-1X7" device=""/>
+<part name="IC1" library="v-reg" deviceset="LP2950?*" device="ACZ" technology="-3.0" value="TS2950-3v3"/>
+<part name="GND1" library="supply1" deviceset="GND" device=""/>
+<part name="P+8" library="supply1" deviceset="+12V" device=""/>
 </parts>
 <sheets>
@@
 <instance part="R2" gate="G$1" x="101.6" y="27.94" rot="R90"/>
 <instance part="R3" gate="G$1" x="91.44" y="48.26" rot="R90"/>
-<instance part="GND1" gate="1" x="2.54" y="63.5"/>
 <instance part="GND2" gate="1" x="111.76" y="83.82"/>
 <instance part="P+1" gate="1" x="-22.86" y="88.9"/>
@@
 <instance part="H4" gate="G$1" x="35.56" y="91.44"/>
 <instance part="GND10" gate="1" x="20.32" y="96.52"/>
-<instance part="IC1" gate="1" x="-12.7" y="81.28" rot="R180"/>
 <instance part="B1" gate="1" x="111.76" y="93.98" smashed="yes" rot="MR90">
 <attribute name="VALUE" x="106.68" y="99.06" size="1.778" layer="96" rot="MR90"/>
 <attribute name="NAME" x="104.14" y="96.52" size="1.778" layer="95" rot="MR180"/>
 </instance>
-<instance part="P+8" gate="VCC" x="-25.4" y="58.42"/>
 <instance part="GND11" gate="1" x="-22.86" y="53.34" rot="R90"/>
 <instance part="JP3" gate="A" x="-38.1" y="48.26" rot="R180"/>
+<instance part="IC1" gate="G$1" x="-12.7" y="81.28"/>
+<instance part="GND1" gate="1" x="2.54" y="63.5"/>
+<instance part="P+8" gate="1" x="-25.4" y="60.96"/>
 </instances>
 <busses>
@@
 <wire x1="-22.86" y1="86.36" x2="-22.86" y2="81.28" width="0.1524" layer="91"/>
 <junction x="-22.86" y="81.28"/>
-<pinref part="IC1" gate="1" pin="OUT"/>
+<pinref part="IC1" gate="G$1" pin="IN"/>
 </segment>
 <segment>
@@
 <junction x="111.76" y="99.06"/>
 </segment>
+<segment>
+<pinref part="JP3" gate="A" pin="7"/>
+<wire x1="-35.56" y1="55.88" x2="-25.4" y2="55.88" width="0.1524" layer="91"/>
+<pinref part="P+8" gate="1" pin="+12V"/>
+<wire x1="-25.4" y1="55.88" x2="-25.4" y2="58.42" width="0.1524" layer="91"/>
+</segment>
 </net>
 <net name="GND" class="0">
@@
 <pinref part="LED3" gate="G$1" pin="C"/>
 <pinref part="GND4" gate="1" pin="GND"/>
-</segment>
-<segment>
-<pinref part="C1" gate="G$1" pin="-"/>
-<wire x1="-27.94" y1="73.66" x2="-27.94" y2="66.04" width="0.1524" layer="91"/>
-<pinref part="GND1" gate="1" pin="GND"/>
-<wire x1="-27.94" y1="66.04" x2="-12.7" y2="66.04" width="0.1524" layer="91"/>
-<wire x1="-12.7" y1="66.04" x2="0" y2="66.04" width="0.1524" layer="91"/>
-<wire x1="0" y1="66.04" x2="2.54" y2="66.04" width="0.1524" layer="91"/>
-<wire x1="2.54" y1="66.04" x2="10.16" y2="66.04" width="0.1524" layer="91"/>
-<pinref part="LED1" gate="G$1" pin="C"/>
-<wire x1="10.16" y1="66.04" x2="20.32" y2="66.04" width="0.1524" layer="91"/>
-<wire x1="20.32" y1="66.04" x2="20.32" y2="73.66" width="0.1524" layer="91"/>
-<wire x1="-12.7" y1="73.66" x2="-12.7" y2="66.04" width="0.1524" layer="91"/>
-<pinref part="C2" gate="G$1" pin="-"/>
-<wire x1="10.16" y1="73.66" x2="10.16" y2="66.04" width="0.1524" layer="91"/>
-<junction x="-12.7" y="66.04"/>
-<junction x="2.54" y="66.04"/>
-<junction x="10.16" y="66.04"/>
-<pinref part="C5" gate="G$1" pin="1"/>
-<wire x1="0" y1="73.66" x2="0" y2="66.04" width="0.1524" layer="91"/>
-<junction x="0" y="66.04"/>
-<pinref part="IC1" gate="1" pin="GND"/>
 </segment>
 <segment>
@@
 <pinref part="GND11" gate="1" pin="GND"/>
 <pinref part="JP3" gate="A" pin="6"/>
+</segment>
+<segment>
+<pinref part="C1" gate="G$1" pin="-"/>
+<wire x1="-27.94" y1="73.66" x2="-27.94" y2="66.04" width="0.1524" layer="91"/>
+<wire x1="-27.94" y1="66.04" x2="-12.7" y2="66.04" width="0.1524" layer="91"/>
+<wire x1="-12.7" y1="66.04" x2="0" y2="66.04" width="0.1524" layer="91"/>
+<wire x1="0" y1="66.04" x2="2.54" y2="66.04" width="0.1524" layer="91"/>
+<pinref part="LED1" gate="G$1" pin="C"/>
+<wire x1="2.54" y1="66.04" x2="10.16" y2="66.04" width="0.1524" layer="91"/>
+<wire x1="10.16" y1="66.04" x2="20.32" y2="66.04" width="0.1524" layer="91"/>
+<wire x1="20.32" y1="66.04" x2="20.32" y2="73.66" width="0.1524" layer="91"/>
+<wire x1="-12.7" y1="73.66" x2="-12.7" y2="66.04" width="0.1524" layer="91"/>
+<pinref part="C2" gate="G$1" pin="-"/>
+<wire x1="10.16" y1="73.66" x2="10.16" y2="66.04" width="0.1524" layer="91"/>
+<junction x="-12.7" y="66.04"/>
+<junction x="10.16" y="66.04"/>
+<pinref part="C5" gate="G$1" pin="1"/>
+<wire x1="0" y1="73.66" x2="0" y2="66.04" width="0.1524" layer="91"/>
+<junction x="0" y="66.04"/>
+<pinref part="IC1" gate="G$1" pin="GND"/>
+<pinref part="GND1" gate="1" pin="GND"/>
+<junction x="2.54" y="66.04"/>
 </segment>
 </net>
@@
 <pinref part="C5" gate="G$1" pin="2"/>
 <junction x="0" y="81.28"/>
-<pinref part="IC1" gate="1" pin="IN"/>
+<pinref part="IC1" gate="G$1" pin="OUT"/>
 </segment>
 <segment>
@@
 <pinref part="P+4" gate="VCC" pin="VCC"/>
 </segment>
-<segment>
-<wire x1="-35.56" y1="55.88" x2="-25.4" y2="55.88" width="0.1524" layer="91"/>
-<pinref part="P+8" gate="VCC" pin="VCC"/>
-<pinref part="JP3" gate="A" pin="7"/>
-</segment>
-</net>
+</net>
