File: WiFi/Electronics/wifiboard.brd (EAGLE design)
At the start: 100 x 41.9 mm, 16 parts, among them IC1 78L05, X1 MKDSN1,5/2-5,08, X2 MKDSN1,5/2-5,08

Commit message: Working on the WiFi/ESP-8266 version...
Parts:
- removed IC1: 78L05, v-reg:78LXX
- removed Q1: (no value), adafruit:SOT23
- added IC2: 7805DT, adafruit:TO252
- added Q2: IPB45N04, transistor-power:D2PACK
- C2: value 47uF -> 1000uF; device rcl:C0805 -> rcl:B45181B
- C3: value 4.7uF -> 1uF
- R1: value 33R -> 27R
- moved C1 35.1 mm to (68.6, 31.8), turned to 270 degrees
- moved R2 24.3 mm to (62.2, 15.2), turned to 90 degrees
- moved C2 13.5 mm to (86.4, 7.62), flipped to the top, turned to 0 degrees
- moved R1 13.3 mm to (86.4, 34.3)
- moved R3 9.92 mm to (50.8, 31.8)
- moved JP1 4.02 mm to (90.2, 29.2), turned to 270 degrees
- moved C3 3.81 mm to (40.6, 35.6)
- moved WEMOS1 2.54 mm to (67.3, 24.1)
Connections:
- removed net N$1: C2.1, IC1.IN, R1.1
- new net N$2: C1.1, IC2.1, R1.1
- net +5V: now also C2.+, IC2.2; no longer C1.1, IC1.OUT
- net GND: now also C2.-, IC2.3, Q2.3; no longer C2.2, IC1.GND, Q1.2
- net N$5: now also Q2.1; no longer Q1.1
- net N$7: now also Q2.2; no longer Q1.3
Routing:
- net N$2: track 0.00 -> 36.4 mm
- net N$4: track 38.8 -> 5.20 mm
- net N$3: track 23.3 -> 48.3 mm
- net N$1: track 7.72 -> 0.00 mm
- net GND: track 90.1 -> 83.5 mm
- net +5V: track 104.7 -> 99.2 mm
- net +12V: track 134.4 -> 129.3 mm
- net N$7: track 26.2 -> 21.1 mm
- net N$15: track 6.35 -> 3.81 mm
- net N$14: track 6.35 -> 3.81 mm
- net N$13: track 6.35 -> 3.81 mm
- net N$11: track 6.35 -> 3.81 mm
- net N$5: track 3.06 -> 3.93 mm
- net N$6: track 10.3 -> 9.72 mm
Other:
- board size 100 x 41.9 mm -> 94.9 x 41.9 mm

Commit message: Improved PCB design and casing.
Parts:
- removed Q2: IPB45N04, transistor-power:D2PACK
- added Q1: FDD8870, SparkFun-DiscreteSemi:DPAK
- C1: value 47uF -> 1000uF; device rcl:C0805 -> rcl:B45181B
- moved C1 22.5 mm to (87.6, 19.7), flipped to the top
- moved IC2 3.81 mm to (63.5, 24.1)
- moved WEMOS1 3.81 mm to (63.5, 24.1)
- moved R2 3.81 mm to (58.4, 15.2)
- moved R3 3.81 mm to (47.0, 31.8)
- moved JP3 3.81 mm to (80.0, 21.6)
- moved R1 3.17 mm to (83.2, 34.3)
- moved C2 0.90 mm to (85.7, 8.26)
Connections:
- net +12V: now also C1.+
- net GND: now also C1.-, Q1.3; no longer C1.2, Q2.3
- net N$2: no longer C1.1
- net N$5: now also Q1.1; no longer Q2.1
- net N$7: now also Q1.4; no longer Q2.2
Routing:
- net +12V: track 129.3 -> 148.4 mm
- net N$7: track 21.1 -> 29.1 mm
- net N$5: track 3.93 -> 9.98 mm
- net N$2: track 36.4 -> 30.4 mm
- net +5V: track 99.2 -> 95.1 mm
- net N$3: track 48.3 -> 44.4 mm
Other:
- board size 94.9 x 41.9 mm -> 95.2 x 43.2 mm
