File: WiFi/Electronics/wifiboard.sch (EAGLE design)
At the start: 16 parts, among them IC1 78L05, X1 MKDSN1,5/2-5,08, X2 MKDSN1,5/2-5,08

Commit message: Working on the WiFi/ESP-8266 version...
Parts:
- removed IC1: 78L05, v-reg:78LXX
- removed Q1: (no value), adafruit:MOSFET-NREFLOW
- added IC2: 7805DT, adafruit:7805DT
- added Q2: IPB45N04, transistor-power:IRF3704S
- C2: value 47uF -> 1000uF; device rcl:C-EUC0805 -> rcl:CPOL-EUB45181B
- C3: value 4.7uF -> 1uF
- R1: value 33R -> 27R
Connections:
- removed net N$1: C2.1, IC1.IN, R1.1
- new net N$2: C1.1, IC2.VI, R1.1
- net +5V: now also C2.+, IC2.VO; no longer C1.1, IC1.OUT
- net GND: now also C2.-, IC2.GND, Q2.S; no longer C2.2, IC1.GND, Q1.S
- net N$5: now also Q2.G; no longer Q1.G
- net N$7: now also Q2.D; no longer Q1.D
Other:
- moved on the sheet: R1
Changed lines of the file:
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@@
 <part name="GND1" library="supply1" deviceset="GND" device=""/>
 <part name="P+1" library="supply1" deviceset="+12V" device=""/>
-<part name="IC1" library="v-reg" deviceset="78LXX" device="" value="78L05"/>
 <part name="C1" library="rcl" deviceset="C-EU" device="C0805" value="47uF"/>
-<part name="C2" library="rcl" deviceset="C-EU" device="C0805" value="47uF"/>
-<part name="R1" library="rcl" deviceset="R-EU_" device="0207/10" value="33R"/>
+<part name="R1" library="rcl" deviceset="R-EU_" device="0207/10" value="27R"/>
 <part name="JP1" library="pinhead" deviceset="PINHD-1X2" device=""/>
 <part name="P+2" library="supply1" deviceset="+12V" device=""/>
@@
 <part name="JP2" library="pinhead" deviceset="PINHD-1X2" device=""/>
 <part name="GND3" library="supply1" deviceset="GND" device=""/>
-<part name="C3" library="rcl" deviceset="C-EU" device="C0805" value="4.7uF"/>
+<part name="C3" library="rcl" deviceset="C-EU" device="C0805" value="1uF"/>
 <part name="R2" library="rcl" deviceset="R-EU_" device="M0805" value="1K"/>
-<part name="Q1" library="adafruit" deviceset="MOSFET-N" device="REFLOW"/>
 <part name="R3" library="rcl" deviceset="R-EU_" device="M0805" value="10K"/>
 <part name="GND4" library="supply1" deviceset="GND" device=""/>
@@
 <part name="P+5" library="supply1" deviceset="+5V" device=""/>
 <part name="U$1" library="alexa" deviceset="OMRON-G6DS" device=""/>
+<part name="IC2" library="adafruit" deviceset="78*" device="DT" technology="05"/>
+<part name="C2" library="rcl" deviceset="CPOL-EU" device="B45181B" value="1000uF"/>
+<part name="Q2" library="transistor-power" deviceset="IRF3704" device="S" value="IPB45N04"/>
 </parts>
 <sheets>
@@
 <instance part="WEMOS1" gate="D1" x="7.62" y="58.42"/>
 <instance part="GND1" gate="1" x="81.28" y="55.88"/>
-<instance part="P+1" gate="1" x="86.36" y="86.36"/>
-<instance part="IC1" gate="1" x="76.2" y="68.58" rot="MR0"/>
+<instance part="P+1" gate="1" x="63.5" y="83.82"/>
 <instance part="C1" gate="G$1" x="60.96" y="66.04"/>
-<instance part="C2" gate="G$1" x="88.9" y="66.04"/>
-<instance part="R1" gate="G$1" x="86.36" y="76.2" rot="R90"/>
+<instance part="R1" gate="G$1" x="63.5" y="76.2" rot="R90"/>
 <instance part="JP1" gate="G$1" x="-25.4" y="15.24"/>
 <instance part="P+2" gate="1" x="-38.1" y="22.86"/>
@@
 <instance part="C3" gate="G$1" x="-22.86" y="43.18"/>
 <instance part="R2" gate="G$1" x="-25.4" y="55.88" rot="R90"/>
-<instance part="Q1" gate="G$1" x="17.78" y="20.32"/>
 <instance part="R3" gate="G$1" x="7.62" y="17.78" rot="R180"/>
 <instance part="GND4" gate="1" x="20.32" y="10.16"/>
@@
 <instance part="JP3" gate="A" x="35.56" y="58.42"/>
 <instance part="GND6" gate="1" x="30.48" y="45.72"/>
-<instance part="P+4" gate="1" x="63.5" y="76.2"/>
+<instance part="P+4" gate="1" x="88.9" y="78.74"/>
 <instance part="P+5" gate="1" x="45.72" y="43.18"/>
 <instance part="U$1" gate="G$1" x="33.02" y="0"/>
+<instance part="IC2" gate="A1" x="76.2" y="68.58"/>
+<instance part="C2" gate="G$1" x="88.9" y="66.04"/>
+<instance part="Q2" gate="G$1" x="17.78" y="20.32"/>
 </instances>
 <busses>
@@
 </segment>
 <segment>
-<pinref part="Q1" gate="G$1" pin="S"/>
 <pinref part="GND4" gate="1" pin="GND"/>
 <wire x1="20.32" y1="15.24" x2="20.32" y2="12.7" width="0.1524" layer="91"/>
+<pinref part="Q2" gate="G$1" pin="S"/>
 </segment>
 <segment>
@@
 </segment>
 <segment>
-<pinref part="IC1" gate="1" pin="GND"/>
 <wire x1="76.2" y1="58.42" x2="76.2" y2="60.96" width="0.1524" layer="91"/>
 <pinref part="C1" gate="G$1" pin="2"/>
 <wire x1="60.96" y1="58.42" x2="76.2" y2="58.42" width="0.1524" layer="91"/>
 <wire x1="60.96" y1="60.96" x2="60.96" y2="58.42" width="0.1524" layer="91"/>
-<pinref part="C2" gate="G$1" pin="2"/>
 <wire x1="76.2" y1="58.42" x2="81.28" y2="58.42" width="0.1524" layer="91"/>
 <wire x1="81.28" y1="58.42" x2="88.9" y2="58.42" width="0.1524" layer="91"/>
@@
 <pinref part="GND1" gate="1" pin="GND"/>
 <junction x="81.28" y="58.42"/>
+<pinref part="IC2" gate="A1" pin="GND"/>
+<pinref part="C2" gate="G$1" pin="-"/>
 </segment>
 <segment>
@@
 </segment>
 </net>
-<net name="N$1" class="0">
-<segment>
-<pinref part="IC1" gate="1" pin="IN"/>
-<pinref part="C2" gate="G$1" pin="1"/>
-<wire x1="88.9" y1="68.58" x2="86.36" y2="68.58" width="0.1524" layer="91"/>
-<pinref part="R1" gate="G$1" pin="1"/>
-<wire x1="86.36" y1="68.58" x2="83.82" y2="68.58" width="0.1524" layer="91"/>
-<wire x1="86.36" y1="71.12" x2="86.36" y2="68.58" width="0.1524" layer="91"/>
-<junction x="86.36" y="68.58"/>
-</segment>
-</net>
 <net name="+12V" class="0">
 <segment>
 <pinref part="R1" gate="G$1" pin="2"/>
 <pinref part="P+1" gate="1" pin="+12V"/>
-<wire x1="86.36" y1="81.28" x2="86.36" y2="83.82" width="0.1524" layer="91"/>
 </segment>
 <segment>
@@
 <net name="N$5" class="0">
 <segment>
-<pinref part="Q1" gate="G$1" pin="G"/>
 <pinref part="R3" gate="G$1" pin="1"/>
 <wire x1="15.24" y1="17.78" x2="12.7" y2="17.78" width="0.1524" layer="91"/>
+<pinref part="Q2" gate="G$1" pin="G"/>
 </segment>
 </net>
@@
 <net name="N$7" class="0">
 <segment>
-<pinref part="Q1" gate="G$1" pin="D"/>
 <wire x1="20.32" y1="27.94" x2="20.32" y2="25.4" width="0.1524" layer="91"/>
 <wire x1="50.8" y1="22.86" x2="50.8" y2="27.94" width="0.1524" layer="91"/>
 <wire x1="50.8" y1="27.94" x2="20.32" y2="27.94" width="0.1524" layer="91"/>
 <pinref part="U$1" gate="G$1" pin="-IN"/>
+<pinref part="Q2" gate="G$1" pin="D"/>
 </segment>
 </net>
@@
 </segment>
 <segment>
-<pinref part="IC1" gate="1" pin="OUT"/>
+<wire x1="88.9" y1="68.58" x2="86.36" y2="68.58" width="0.1524" layer="91"/>
+<pinref part="IC2" gate="A1" pin="VO"/>
+<pinref part="P+4" gate="1" pin="+5V"/>
+<wire x1="88.9" y1="76.2" x2="88.9" y2="68.58" width="0.1524" layer="91"/>
+<pinref part="C2" gate="G$1" pin="+"/>
+<junction x="88.9" y="68.58"/>
+</segment>
+</net>
+<net name="N$2" class="0">
+<segment>
 <pinref part="C1" gate="G$1" pin="1"/>
-<wire x1="60.96" y1="68.58" x2="63.5" y2="68.58" width="0.1524" layer="91"/>
-<pinref part="P+4" gate="1" pin="+5V"/>
-<wire x1="63.5" y1="68.58" x2="68.58" y2="68.58" width="0.1524" layer="91"/>
-<wire x1="63.5" y1="73.66" x2="63.5" y2="68.58" width="0.1524" layer="91"/>
+<pinref part="IC2" gate="A1" pin="VI"/>
+<wire x1="66.04" y1="68.58" x2="63.5" y2="68.58" width="0.1524" layer="91"/>
+<pinref part="R1" gate="G$1" pin="1"/>
+<wire x1="63.5" y1="68.58" x2="60.96" y2="68.58" width="0.1524" layer="91"/>
+<wire x1="63.5" y1="71.12" x2="63.5" y2="68.58" width="0.1524" layer="91"/>
 <junction x="63.5" y="68.58"/>
 </segment>

Commit message: Improved PCB design and casing.
Parts:
- removed Q2: IPB45N04, transistor-power:IRF3704S
- added Q1: FDD8870, SparkFun-DiscreteSemi:MOSFET-NCH-FDD8780
- C1: value 47uF -> 1000uF; device rcl:C-EUC0805 -> rcl:CPOL-EUB45181B
Connections:
- net +12V: now also C1.+
- net GND: now also C1.-, Q1.S; no longer C1.2, Q2.S
- net N$2: no longer C1.1
- net N$5: now also Q1.G; no longer Q2.G
- net N$7: now also Q1.D; no longer Q2.D
Changed lines of the file:
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@@
 <layer number="112" name="tSilk" color="7" fill="1" visible="no" active="yes"/>
 <layer number="113" name="ReferenceLS" color="7" fill="1" visible="no" active="no"/>
+<layer number="114" name="Badge_Outline" color="7" fill="1" visible="yes" active="yes"/>
+<layer number="115" name="ReferenceISLANDS" color="7" fill="1" visible="yes" active="yes"/>
 <layer number="116" name="Patch_BOT" color="9" fill="4" visible="no" active="yes"/>
 <layer number="118" name="Rect_Pads" color="7" fill="1" visible="no" active="no"/>
@@
 <part name="GND1" library="supply1" deviceset="GND" device=""/>
 <part name="P+1" library="supply1" deviceset="+12V" device=""/>
-<part name="C1" library="rcl" deviceset="C-EU" device="C0805" value="47uF"/>
 <part name="R1" library="rcl" deviceset="R-EU_" device="0207/10" value="27R"/>
 <part name="JP1" library="pinhead" deviceset="PINHD-1X2" device=""/>
@@
 <part name="IC2" library="adafruit" deviceset="78*" device="DT" technology="05"/>
 <part name="C2" library="rcl" deviceset="CPOL-EU" device="B45181B" value="1000uF"/>
-<part name="Q2" library="transistor-power" deviceset="IRF3704" device="S" value="IPB45N04"/>
+<part name="Q1" library="SparkFun-DiscreteSemi" deviceset="MOSFET-NCH" device="-FDD8780" value="FDD8870"/>
+<part name="C1" library="rcl" deviceset="CPOL-EU" device="B45181B" value="1000uF"/>
 </parts>
 <sheets>
@@
 <instance part="GND1" gate="1" x="81.28" y="55.88"/>
 <instance part="P+1" gate="1" x="63.5" y="83.82"/>
-<instance part="C1" gate="G$1" x="60.96" y="66.04"/>
 <instance part="R1" gate="G$1" x="63.5" y="76.2" rot="R90"/>
 <instance part="JP1" gate="G$1" x="-25.4" y="15.24"/>
@@
 <instance part="R2" gate="G$1" x="-25.4" y="55.88" rot="R90"/>
 <instance part="R3" gate="G$1" x="7.62" y="17.78" rot="R180"/>
-<instance part="GND4" gate="1" x="20.32" y="10.16"/>
+<instance part="GND4" gate="1" x="22.86" y="10.16"/>
 <instance part="U$2" gate="G$1" x="73.66" y="27.94"/>
 <instance part="X1" gate="-1" x="93.98" y="7.62"/>
@@
 <instance part="IC2" gate="A1" x="76.2" y="68.58"/>
 <instance part="C2" gate="G$1" x="88.9" y="66.04"/>
-<instance part="Q2" gate="G$1" x="17.78" y="20.32"/>
+<instance part="Q1" gate="NMOS" x="20.32" y="20.32"/>
+<instance part="C1" gate="G$1" x="60.96" y="66.04"/>
 </instances>
 <busses>
@@
 <segment>
 <pinref part="GND4" gate="1" pin="GND"/>
-<wire x1="20.32" y1="15.24" x2="20.32" y2="12.7" width="0.1524" layer="91"/>
-<pinref part="Q2" gate="G$1" pin="S"/>
+<wire x1="22.86" y1="15.24" x2="22.86" y2="12.7" width="0.1524" layer="91"/>
+<pinref part="Q1" gate="NMOS" pin="S"/>
+<junction x="22.86" y="15.24"/>
 </segment>
 <segment>
@@
 <segment>
 <wire x1="76.2" y1="58.42" x2="76.2" y2="60.96" width="0.1524" layer="91"/>
-<pinref part="C1" gate="G$1" pin="2"/>
 <wire x1="60.96" y1="58.42" x2="76.2" y2="58.42" width="0.1524" layer="91"/>
 <wire x1="60.96" y1="60.96" x2="60.96" y2="58.42" width="0.1524" layer="91"/>
@@
 <pinref part="IC2" gate="A1" pin="GND"/>
 <pinref part="C2" gate="G$1" pin="-"/>
+<pinref part="C1" gate="G$1" pin="-"/>
 </segment>
 <segment>
@@
 <pinref part="R1" gate="G$1" pin="2"/>
 <pinref part="P+1" gate="1" pin="+12V"/>
+<pinref part="C1" gate="G$1" pin="+"/>
+<wire x1="63.5" y1="81.28" x2="60.96" y2="81.28" width="0.1524" layer="91"/>
+<wire x1="60.96" y1="81.28" x2="60.96" y2="68.58" width="0.1524" layer="91"/>
 </segment>
 <segment>
@@
 <pinref part="R3" gate="G$1" pin="1"/>
 <wire x1="15.24" y1="17.78" x2="12.7" y2="17.78" width="0.1524" layer="91"/>
-<pinref part="Q2" gate="G$1" pin="G"/>
+<pinref part="Q1" gate="NMOS" pin="G"/>
+<junction x="15.24" y="17.78"/>
 </segment>
 </net>
@@
 <net name="N$7" class="0">
 <segment>
-<wire x1="20.32" y1="27.94" x2="20.32" y2="25.4" width="0.1524" layer="91"/>
+<wire x1="22.86" y1="27.94" x2="22.86" y2="25.4" width="0.1524" layer="91"/>
 <wire x1="50.8" y1="22.86" x2="50.8" y2="27.94" width="0.1524" layer="91"/>
-<wire x1="50.8" y1="27.94" x2="20.32" y2="27.94" width="0.1524" layer="91"/>
+<wire x1="50.8" y1="27.94" x2="22.86" y2="27.94" width="0.1524" layer="91"/>
 <pinref part="U$1" gate="G$1" pin="-IN"/>
-<pinref part="Q2" gate="G$1" pin="D"/>
+<pinref part="Q1" gate="NMOS" pin="D"/>
+<junction x="22.86" y="25.4"/>
 </segment>
 </net>
@@
 <net name="N$2" class="0">
 <segment>
-<pinref part="C1" gate="G$1" pin="1"/>
 <pinref part="IC2" gate="A1" pin="VI"/>
 <wire x1="66.04" y1="68.58" x2="63.5" y2="68.58" width="0.1524" layer="91"/>
 <pinref part="R1" gate="G$1" pin="1"/>
-<wire x1="63.5" y1="68.58" x2="60.96" y2="68.58" width="0.1524" layer="91"/>
 <wire x1="63.5" y1="71.12" x2="63.5" y2="68.58" width="0.1524" layer="91"/>
-<junction x="63.5" y="68.58"/>
-</segment>
-</net>
+</segment>
+</net>
