File: ESP-8266/Electronics/KiCAD/wifiboard-v2.sch (KiCad schematic (older format))
At the start: 30 parts, among them IC2 78033AF, Q1 FDD8870, U2 ESP12ESMD, X1 AC-N, X2 AC-L

Commit message: Tidying files; previous...
Connections:
- net at R10.2: now also U2.GPIO4
Other:
- moved on the sheet: LED2, R10
Changed lines of the file:
@@
 $EndComp
 Wire Wire Line
-	2500 6400 2500 6500
+	4950 6475 4950 6575
 $Comp
 L wifiboard-v2-eagle-import:R-EU_R0805 R10
 U 1 1 6080063F
-P 2500 6200
-F 0 "R10" H 2350 6259 59  0000 L BNN
-F 1 "180R" H 2350 6070 59  0000 L BNN
-F 2 "wifiboard-v2:R0805" H 2500 6200 50  0001 C CNN
-F 3 "" H 2500 6200 50  0001 C CNN
-	1    2500 6200
+P 4950 6275
+F 0 "R10" H 4800 6334 59  0000 L BNN
+F 1 "180R" H 4800 6145 59  0000 L BNN
+F 2 "wifiboard-v2:R0805" H 4950 6275 50  0001 C CNN
+F 3 "" H 4950 6275 50  0001 C CNN
+	1    4950 6275
 	0    -1   -1   0
 $EndComp
@@
 L wifiboard-v2-eagle-import:LED3MM LED2
 U 1 1 60800645
-P 2500 6600
-F 0 "LED2" V 2640 6420 59  0000 L BNN
-F 1 "LED3MM" V 2725 6420 59  0000 L BNN
-F 2 "wifiboard-v2:LED3MM" H 2500 6600 50  0001 C CNN
-F 3 "" H 2500 6600 50  0001 C CNN
-	1    2500 6600
+P 4950 6675
+F 0 "LED2" V 5090 6495 59  0000 L BNN
+F 1 "LED3MM" V 5175 6495 59  0000 L BNN
+F 2 "wifiboard-v2:LED3MM" H 4950 6675 50  0001 C CNN
+F 3 "" H 4950 6675 50  0001 C CNN
+	1    4950 6675
+	1    0    0    -1
+$EndComp
+$Comp
+L wifiboard-v2-eagle-import:GND #GND0101
+U 1 1 60806A8D
+P 4950 7175
+F 0 "#GND0101" H 4950 7175 50  0001 C CNN
+F 1 "GND" H 4850 7075 59  0000 L BNN
+F 2 "" H 4950 7175 50  0001 C CNN
+F 3 "" H 4950 7175 50  0001 C CNN
+	1    4950 7175
 	1    0    0    -1
 $EndComp
 Wire Wire Line
-	2500 5875 2500 6000
-$Comp
-L wifiboard-v2-eagle-import:GND #GND0101
-U 1 1 60806A8D
-P 2500 7100
-F 0 "#GND0101" H 2500 7100 50  0001 C CNN
-F 1 "GND" H 2400 7000 59  0000 L BNN
-F 2 "" H 2500 7100 50  0001 C CNN
-F 3 "" H 2500 7100 50  0001 C CNN
-	1    2500 7100
-	1    0    0    -1
-$EndComp
+	4950 6875 4950 7075
 Wire Wire Line
-	2500 6800 2500 7000
+	4900 4500 4950 4500
+Wire Wire Line
+	4950 4500 4950 6075
 $EndSCHEMATC
