File: ESP-8266/Electronics/KiCAD/V4-Design/wifiboard-v4.sch (KiCad schematic (older format))
At the start: 33 parts, among them IC2 78033AF, J1 Conn_01x07_Male, J2 Conn_01x03_Male, Q1 FDD8870, U2 ESP12ESMD

Commit message: Redoing V4 electronics to make it fully KiCAD.
Parts:
- removed 12V-IN1, PROG1, THERMISTOR1: PINHD-1X2, wifiboard-v2:1X02, symbol wifiboard-v3-rescue:PINHD-1X2-wifiboard-v2-eagle-import
- removed C1, C2: 1000uF, wifiboard-v2:B45181B, symbol wifiboard-v3-rescue:CPOL-EUB45181B-wifiboard-v2-eagle-import
- removed C3: 1uF, wifiboard-v2:C0805, symbol wifiboard-v3-rescue:C-EUC0805-wifiboard-v2-eagle-import
- removed C5, C6: 0.1u, wifiboard-v2:C0805, symbol wifiboard-v3-rescue:C-EUC0805-wifiboard-v2-eagle-import
- removed GPIO1: PINHD-1X5, wifiboard-v2:1X05, symbol wifiboard-v3-rescue:PINHD-1X5-wifiboard-v2-eagle-import
- removed H1, H2, H3, H4: MountingHole, MountingHole:MountingHole_2.5mm, symbol Mechanical:MountingHole
- removed IC2: 78033AF, wifiboard-v2:TO252, symbol wifiboard-v3-rescue:78DT-wifiboard-v2-eagle-import
- removed J1: Conn_01x07_Male, Connector_PinHeader_2.54mm:PinHeader_1x07_P2.54mm_Vertical, symbol Connector:Conn_01x07_Male
- removed J2: Conn_01x03_Male, Connector_PinHeader_2.54mm:PinHeader_1x03_P2.54mm_Vertical, symbol Connector:Conn_01x03_Male
- removed LED1, LED2: LED3MM, wifiboard-v2:LED3MM, symbol wifiboard-v3-rescue:LED3MM-wifiboard-v2-eagle-import
- removed Q1: FDD8870, wifiboard-v2:DPAK, symbol wifiboard-v3-rescue:MOSFET-NCH-FDD8780-wifiboard-v2-eagle-import
- removed R1: 6R8, wifiboard-v2:0207_10, symbol wifiboard-v3-rescue:R-EU_0207_10-wifiboard-v2-eagle-import
- removed R10: 180R, wifiboard-v2:R0805, symbol wifiboard-v3-rescue:R-EU_R0805-wifiboard-v2-eagle-import
- removed R2, R3: 10K, wifiboard-v2:M0805, symbol wifiboard-v3-rescue:R-EU_M0805-wifiboard-v2-eagle-import
- removed R4, R5, R6, R7, R8: 10K, wifiboard-v2:R0805, symbol wifiboard-v3-rescue:R-EU_R0805-wifiboard-v2-eagle-import
- removed R9: 1K, wifiboard-v2:R0805, symbol wifiboard-v3-rescue:R-EU_R0805-wifiboard-v2-eagle-import
- removed RESET1: (no value), wifiboard-v2:TACTILE_SWITCH_SMD_4.6X2.8MM, symbol wifiboard-v3-rescue:MOMENTARY-SWITCH-SPST-SMD-4.6X2.8MM-wifiboard-v2-eagle-impo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
- removed RLA1: OMRON-G6DN, wifiboard-v2:OMRON-G6DN-1A, symbol wifiboard-v3-rescue:OMRON-G6DN-wifiboard-v2-eagle-import
- removed U2: ESP12ESMD, wifiboard-v2:ESP12E-SMD, symbol wifiboard-v3-rescue:ESP12ESMD-wifiboard-v2-eagle-import
- removed USB-3V3: PINHD-1X6, wifiboard-v2:1X06, symbol wifiboard-v3-rescue:PINHD-1X6-wifiboard-v2-eagle-import
- added C? (x3): 0.1u, Capacitor_SMD:C_0805_2012Metric, symbol Device:C
- added C? (x2): 1000u, Capacitor_THT:CP_Radial_D10.0mm_P5.00mm, symbol Device:CP
- added D? (x2): LED, LED_THT:LED_D3.0mm, symbol Device:LED
- added IC?: 78033AF, Package_TO_SOT_SMD:TO-252-2, symbol adafruit-new:7805DT
- added J?: USB-3V3, Connector_PinHeader_2.54mm:PinHeader_1x06_P2.54mm_Vertical, symbol Connector:Conn_01x06_Male
- added J?: Aux1, Connector_PinHeader_2.54mm:PinHeader_1x05_P2.54mm_Vertical, symbol Connector:Conn_01x05_Male
- added J?: Aux2, Connector_PinHeader_2.54mm:PinHeader_1x07_P2.54mm_Vertical, symbol Connector:Conn_01x07_Male
- added J?: thermistor, Connector_PinHeader_2.54mm:PinHeader_1x02_P2.54mm_Vertical, symbol Connector:Conn_01x02_Male
- added J?: PWR, Connector_PinHeader_2.54mm:PinHeader_1x02_P2.54mm_Vertical, symbol Connector:Conn_01x02_Male
- added J?: PROG, Connector_PinHeader_2.54mm:PinHeader_1x02_P2.54mm_Vertical, symbol Connector:Conn_01x02_Male
- added J?: Conn_01x03_Male, symbol Connector:Conn_01x03_Male
- added K?: SIL12-1A72-71L, Relay_THT:Relay_SPST_StandexMeder_SIL_Form1A, symbol Relay:SILxx-1Axx-71x
- added Q?: FDD8870, Package_TO_SOT_SMD:TO-252-2, symbol Transistor_FET:FDMS8350L
- added R?: 6R8, Resistor_THT:R_Axial_DIN0414_L11.9mm_D4.5mm_P15.24mm_Horizontal, symbol Device:R
- added R? (x7): 10K, Resistor_SMD:R_0805_2012Metric, symbol Device:R
- added R?: 180R, Resistor_SMD:R_0805_2012Metric, symbol Device:R
- added R?: 1K, Resistor_SMD:R_0805_2012Metric, symbol Device:R
- added SW?: reset, Button_Switch_SMD:SW_SPST_TL3342, symbol Switch:SW_Push
- added U?: ESP-12E, esp-8266:ESP-12E, symbol esp-8266:ESP-12E
Connections:
- net labels added: +3.3V
- net labels removed: +3V3
- wire segments 106 -> 105
Other:
- note removed: "10K gives a min. \ntemp of -9 C."
- note removed: "Max 1V."
- note removed: "relay"

Commit message: V4 schematic complete (?)...
Parts:
- removed K?: SIL12-1A72-71L, Relay_THT:Relay_SPST_StandexMeder_SIL_Form1A, symbol Relay:SILxx-1Axx-71x
- added J?: mains, TerminalBlock:TerminalBlock_bornier-2_P5.08mm, symbol Connector:Screw_Terminal_01x02
- added K?: CPC1966Y, reprapltd-kicad:CPC1966Y, symbol cpc1966y:CPC1966Y
- added R?: 1K, Resistor_SMD:R_0805_2012Metric, symbol Device:R
- J?: value Conn_01x03_Male -> OUT; footprint (none) -> Connector_PinHeader_2.54mm:PinHeader_1x03_P2.54mm_Vertical
Connections:
- wire segments 105 -> 108
Other:
- moved on the sheet: J?
Changed lines of the file:
@@
 	1    0    0    -1
 $EndComp
-Wire Wire Line
-	7475 4275 7475 4325
 Connection ~ 5675 5100
 Wire Wire Line
@@
 	1    0    0    -1
 $EndComp
-Wire Wire Line
-	7475 2975 7475 3025
 $Comp
 L Connector:Conn_01x03_Male J?
 U 1 1 620106EE
-P 8975 3850
-F 0 "J?" H 8947 3782 50  0000 R CNN
-F 1 "Conn_01x03_Male" H 8947 3873 50  0000 R CNN
-F 2 "" H 8975 3850 50  0001 C CNN
-F 3 "~" H 8975 3850 50  0001 C CNN
-	1    8975 3850
+P 8200 3850
+F 0 "J?" H 8172 3782 50  0000 R CNN
+F 1 "OUT" H 8172 3873 50  0000 R CNN
+F 2 "Connector_PinHeader_2.54mm:PinHeader_1x03_P2.54mm_Vertical" H 8200 3850 50  0001 C CNN
+F 3 "~" H 8200 3850 50  0001 C CNN
+	1    8200 3850
 	-1   0    0    1
 $EndComp
-Connection ~ 7475 3025
 Wire Wire Line
-	7475 3025 7475 3075
-Wire Wire Line
-	7475 4325 8775 4325
-Wire Wire Line
-	8775 4325 8775 3950
-Connection ~ 7475 4325
-Wire Wire Line
-	7475 4325 7475 4400
+	8000 4325 8000 3950
 Wire Wire Line
 	6075 3600 6075 3700
@@
 	5675 3600 5675 4400
 Wire Wire Line
-	7475 3025 7825 3025
+	7475 3750 7475 3850
 Wire Wire Line
-	8775 3025 8775 3450
+	8000 3025 8000 3475
 Wire Wire Line
-	7475 3750 7475 3800
+	7475 2975 7475 3025
+Wire Wire Line
+	7475 4275 7475 4325
+Wire Wire Line
+	8000 3025 7475 3025
+Connection ~ 7475 3025
+Wire Wire Line
+	7475 3025 7475 3075
+Wire Wire Line
+	8000 3850 7775 3850
+Connection ~ 7475 3850
+Wire Wire Line
+	7475 3850 7475 3875
+Wire Wire Line
+	8000 4325 7475 4325
+Connection ~ 7475 4325
+Wire Wire Line
+	7475 4325 7475 4400
 $Comp
-L Relay:SILxx-1Axx-71x K?
-U 1 1 6204C4EE
-P 8275 3650
-F 0 "K?" V 7708 3650 50  0000 C CNN
-F 1 "SIL12-1A72-71L" V 7799 3650 50  0000 C CNN
-F 2 "Relay_THT:Relay_SPST_StandexMeder_SIL_Form1A" H 8625 3600 50  0001 L CNN
-F 3 "https://standexelectronics.com/wp-content/uploads/datasheet_reed_relay_SIL.pdf" H 8275 3650 50  0001 C CNN
-	1    8275 3650
-	0    1    1    0
+L cpc1966y:CPC1966Y K?
+U 1 1 61FAC409
+P 8275 3075
+F 0 "K?" V 8813 2647 50  0000 R CNN
+F 1 "CPC1966Y" V 8722 2647 50  0000 R CNN
+F 2 "reprapltd-kicad:CPC1966Y" H 9325 3175 50  0001 L CNN
+F 3 "https://datasheet.datasheetarchive.com/originals/distributors/Datasheets_SAMA/4bd38bcd53ac06cbf93d43ee226943fd.pdf" H 9325 3075 50  0001 L CNN
+F 4 "IXYS 3 A rms SPNO Solid State Relay, Zero Crossing, PCB Mount SCR, 240 V ac Maximum Load" H 9325 2975 50  0001 L CNN "Description"
+F 5 "10" H 9325 2875 50  0001 L CNN "Height"
+F 6 "LITTELFUSE" H 9325 2775 50  0001 L CNN "Manufacturer_Name"
+F 7 "CPC1966Y" H 9325 2675 50  0001 L CNN "Manufacturer_Part_Number"
+F 8 "849-CPC1966Y" H 9325 2575 50  0001 L CNN "Mouser Part Number"
+F 9 "https://www.mouser.co.uk/ProductDetail/IXYS-Integrated-Circuits/CPC1966Y?qs=8uBHJDVwVqxNfAOiNv29Iw%3D%3D" H 9325 2475 50  0001 L CNN "Mouser Price/Stock"
+F 10 "CPC1966Y" H 9325 2375 50  0001 L CNN "Arrow Part Number"
+F 11 "https://www.arrow.com/en/products/cpc1966y/ixys" H 9325 2275 50  0001 L CNN "Arrow Price/Stock"
+	1    8275 3075
+	0    -1   -1   0
+$EndComp
+$Comp
+L Device:R R?
+U 1 1 61FAD78C
+P 8375 3325
+F 0 "R?" H 8445 3371 50  0000 L CNN
+F 1 "1K" H 8445 3280 50  0000 L CNN
+F 2 "Resistor_SMD:R_0805_2012Metric" V 8305 3325 50  0001 C CNN
+F 3 "~" H 8375 3325 50  0001 C CNN
+	1    8375 3325
+	1    0    0    -1
 $EndComp
 Wire Wire Line
-	8575 3450 8775 3450
-Connection ~ 8775 3450
+	8375 3075 8375 3175
 Wire Wire Line
-	8775 3450 8775 3750
+	8375 3475 8000 3475
+Connection ~ 8000 3475
 Wire Wire Line
-	7975 3450 7675 3450
+	8000 3475 8000 3750
 Wire Wire Line
-	7675 3450 7675 3800
+	8275 3075 8275 3250
 Wire Wire Line
-	7675 3800 7475 3800
-Connection ~ 7475 3800
+	8275 3250 7775 3250
 Wire Wire Line
-	7475 3800 7475 3875
+	7775 3250 7775 3850
+Connection ~ 7775 3850
 Wire Wire Line
-	7975 3850 7825 3850
+	7775 3850 7475 3850
+$Comp
+L Connector:Screw_Terminal_01x02 J?
+U 1 1 61FBF554
+P 9275 3125
+F 0 "J?" H 9355 3117 50  0000 L CNN
+F 1 "mains" H 9355 3026 50  0000 L CNN
+F 2 "TerminalBlock:TerminalBlock_bornier-2_P5.08mm" H 9275 3125 50  0001 C CNN
+F 3 "~" H 9275 3125 50  0001 C CNN
+	1    9275 3125
+	1    0    0    -1
+$EndComp
 Wire Wire Line
-	7825 3850 7825 3025
-Connection ~ 7825 3025
+	9075 3125 8575 3125
 Wire Wire Line
-	7825 3025 8775 3025
+	8575 3125 8575 3075
 Wire Wire Line
-	8575 3850 8775 3850
+	8475 3075 8475 3225
+Wire Wire Line
+	8475 3225 9075 3225
 $EndSCHEMATC

Commit message: Components positioned on PCB.
Parts:
- removed Q?: FDD8870, Package_TO_SOT_SMD:TO-252-2, symbol Transistor_FET:FDMS8350L
- added H1, H2, H3, H4: MountingHole, MountingHole:MountingHole_2.5mm, symbol Mechanical:MountingHole
- added J10, J9: Conn_01x01_Male, Connector_PinHeader_2.54mm:PinHeader_1x01_P2.54mm_Vertical, symbol Connector:Conn_01x01_Male
- added Q1: FDD8870, Package_TO_SOT_SMD:TO-252-2, symbol Transistor_FET:QM6006D
- C2: renamed from C?; value 0.1u -> 1u
- R10: renamed from R?; value 1K -> 180R
- gave numbers to parts that had none: 28
Connections:
- wire segments 108 -> 107
Other:
- moved on the sheet: D2, R10

Commit message: SB & AB PCB layout
Parts:
- removed IC1: 78033AF, Package_TO_SOT_SMD:TO-252-2, symbol adafruit-new:7805DT
- removed J10, J9: Conn_01x01_Male, Connector_PinHeader_2.54mm:PinHeader_1x01_P2.54mm_Vertical, symbol Connector:Conn_01x01_Male
- added J9: led-select, Connector_PinHeader_2.54mm:PinHeader_1x02_P2.54mm_Vertical, symbol Connector:Conn_01x02_Male
- added U2: 78033, Package_TO_SOT_SMD:TO-252-2, symbol Regulator_Linear:L7805
Connections:
- net +3V3: now also U2.3 (OUT)
- net GND: now also U2.2 (GND)
- net at R9.2, U1.14 (GPIO5): now also J9.2 (Pin_2)
- net at C1.1, R1.2: now also U2.1 (IN)
- net at R10.1: now also J9.1 (Pin_1)
Changed lines of the file:
@@
 	4000 3575 4000 3600
-$Comp
-L adafruit-new:7805DT IC1
-U 1 1 61F84DB3
-P 2500 3300
-F 0 "IC1" H 2500 3554 45  0000 C CNN
-F 1 "78033AF" H 2500 3470 45  0000 C CNN
-F 2 "Package_TO_SOT_SMD:TO-252-2" H 2530 3450 20  0001 C CNN
-F 3 "" H 2500 3300 50  0001 C CNN
-	1    2500 3300
-	1    0    0    -1
-$EndComp
 $Comp
 L Device:R R1
@@
 $EndComp
 Wire Wire Line
-	2100 3300 1900 3300
-Wire Wire Line
 	1900 3300 1900 3275
 $Comp
@@
 	1    0    0    -1
 $EndComp
-Wire Wire Line
-	2500 3600 2500 3625
 $Comp
 L power:+12V #PWR0110
@@
 Wire Wire Line
 	1300 3625 1900 3625
-Connection ~ 2500 3625
-Wire Wire Line
-	2500 3625 2500 3650
 $Comp
 L power:+3.3V #PWR0111
@@
 	1    0    0    -1
 $EndComp
-Wire Wire Line
-	2900 3300 3000 3300
 $Comp
 L Device:CP C1
@@
 	1    0    0    -1
 $EndComp
-Connection ~ 1900 3625
-Wire Wire Line
-	1900 3625 2500 3625
 Wire Wire Line
 	1900 3300 1900 3325
 Connection ~ 1900 3300
-Wire Wire Line
-	3000 3650 2500 3650
-Connection ~ 2500 3650
-Wire Wire Line
-	2500 3650 2500 3675
 Wire Wire Line
 	3000 3350 3000 3300
@@
 Wire Wire Line
 	5675 4600 6050 4600
-Wire Wire Line
-	6050 4075 6625 4075
 $Comp
 L Device:R R9
@@
 Wire Wire Line
 	7025 5700 7025 5825
-$Comp
-L Connector:Conn_01x01_Male J10
-U 1 1 62042A4C
-P 7025 4725
-F 0 "J10" V 7087 4769 50  0000 L CNN
-F 1 "Conn_01x01_Male" V 7178 4769 50  0000 L CNN
-F 2 "Connector_PinHeader_2.54mm:PinHeader_1x01_P2.54mm_Vertical" H 7025 4725 50  0001 C CNN
-F 3 "~" H 7025 4725 50  0001 C CNN
-	1    7025 4725
-	0    1    1    0
-$EndComp
 Wire Wire Line
 	7025 4925 7025 5000
 $Comp
-L Connector:Conn_01x01_Male J9
-U 1 1 62057289
-P 6625 3875
-F 0 "J9" V 6687 3919 50  0000 L CNN
-F 1 "Conn_01x01_Male" V 6778 3919 50  0000 L CNN
-F 2 "Connector_PinHeader_2.54mm:PinHeader_1x01_P2.54mm_Vertical" H 6625 3875 50  0001 C CNN
-F 3 "~" H 6625 3875 50  0001 C CNN
-	1    6625 3875
-	0    1    1    0
-$EndComp
-Connection ~ 6625 4075
-Wire Wire Line
-	6625 4075 6775 4075
+L Connector:Conn_01x02_Male J9
+U 1 1 61FC195B
+P 7100 4550
+F 0 "J9" H 7208 4731 50  0000 C CNN
+F 1 "led-select" H 7208 4640 50  0000 C CNN
+F 2 "Connector_PinHeader_2.54mm:PinHeader_1x02_P2.54mm_Vertical" H 7100 4550 50  0001 C CNN
+F 3 "~" H 7100 4550 50  0001 C CNN
+	1    7100 4550
+	-1   0    0    1
+$EndComp
+Wire Wire Line
+	6050 4075 6675 4075
+Wire Wire Line
+	6675 4075 6675 4450
+Wire Wire Line
+	6675 4450 6900 4450
+Connection ~ 6675 4075
+Wire Wire Line
+	6675 4075 6775 4075
+Wire Wire Line
+	7025 4925 6900 4925
+Wire Wire Line
+	6900 4925 6900 4550
+$Comp
+L Regulator_Linear:L7805 U2
+U 1 1 61FDBAF2
+P 2500 3300
+F 0 "U2" H 2500 3542 50  0000 C CNN
+F 1 "78033" H 2500 3451 50  0000 C CNN
+F 2 "Package_TO_SOT_SMD:TO-252-2" H 2525 3150 50  0001 L CIN
+F 3 "http://www.st.com/content/ccc/resource/technical/document/datasheet/41/4f/b3/b0/12/d4/47/88/CD00000444.pdf/files/CD00000444.pdf/jcr:content/translations/en.CD00000444.pdf" H 2500 3250 50  0001 C CNN
+	1    2500 3300
+	1    0    0    -1
+$EndComp
+Wire Wire Line
+	1900 3300 2200 3300
+Wire Wire Line
+	2800 3300 3000 3300
+Wire Wire Line
+	2500 3600 2500 3625
+Wire Wire Line
+	3000 3650 2500 3650
+Connection ~ 2500 3650
+Wire Wire Line
+	2500 3650 2500 3675
+Wire Wire Line
+	1900 3625 2500 3625
+Connection ~ 1900 3625
+Connection ~ 2500 3625
+Wire Wire Line
+	2500 3625 2500 3650
 $EndSCHEMATC

Commit message: PCB sent for trial production.
Parts:
- added JP1: SolderJumper_2_Bridged, Jumper:SolderJumper-2_P1.3mm_Bridged_RoundedPad1.0x1.5mm, symbol Jumper:SolderJumper_2_Bridged
- K1: symbol cpc1966y:CPC1966Y -> wifiboard-v4-rescue:CPC1966Y-cpc1966y
- U1: symbol esp-8266:ESP-12E -> wifiboard-v4-rescue:ESP-12E-esp-8266
Connections:
- net at J9.2 (Pin_2), R9.2, U1.14 (GPIO5): now also JP1.1 (A)
- net at J9.1 (Pin_1), R10.1: now also JP1.2 (B)
Changed lines of the file:
@@
 $EndComp
 $Comp
-L esp-8266:ESP-12E U1
+L wifiboard-v4-rescue:ESP-12E-esp-8266 U1
 U 1 1 61F7D88E
 P 4775 4700
@@
 	7475 4325 7475 4400
 $Comp
-L cpc1966y:CPC1966Y K1
+L wifiboard-v4-rescue:CPC1966Y-cpc1966y K1
 U 1 1 61FAC409
 P 8275 3075
@@
 	6675 4075 6675 4450
 Wire Wire Line
-	6675 4450 6900 4450
+	6675 4450 6725 4450
 Connection ~ 6675 4075
 Wire Wire Line
@@
 	7025 4925 6900 4925
 Wire Wire Line
-	6900 4925 6900 4550
+	6900 4925 6900 4750
 $Comp
 L Regulator_Linear:L7805 U2
@@
 Wire Wire Line
 	2500 3625 2500 3650
+$Comp
+L Jumper:SolderJumper_2_Bridged JP1
+U 1 1 61FD9520
+P 6725 4600
+F 0 "JP1" V 6679 4668 50  0000 L CNN
+F 1 "SolderJumper_2_Bridged" V 6770 4668 50  0000 L CNN
+F 2 "Jumper:SolderJumper-2_P1.3mm_Bridged_RoundedPad1.0x1.5mm" H 6725 4600 50  0001 C CNN
+F 3 "~" H 6725 4600 50  0001 C CNN
+	1    6725 4600
+	0    1    1    0
+$EndComp
+Connection ~ 6725 4450
+Wire Wire Line
+	6725 4450 6900 4450
+Wire Wire Line
+	6725 4750 6900 4750
+Connection ~ 6900 4750
+Wire Wire Line
+	6900 4750 6900 4550
 $EndSCHEMATC
